File: kicad_boilermon/kicad_boilermon.kicad_sch (KiCad schematic)
At the start: 28 parts, among them U1 ESP32-S2-DevKitC-1, U11 PC847, U12 PCF8574, U2 DS18B20, U3 DS18B20, U4 DS18B20, U5 DS18B20, U6 DS18B20, U7 DS18B20, U8 LM2596T-ADJ

Commit message: new sketch, updated readme
Parts:
- removed C2, C3: 10uF, symbol Device:C_Polarized
- removed R12: 6.8k, symbol Device:R
- removed R3, R4, R5, R6: 4.7k, symbol Device:R
- removed U1: ESP32-S2-DevKitC-1, PCM_Espressif:ESP32-S2-DevKitC-1, symbol PCM_Espressif:ESP32-S2-DevKitC-1
- removed U12: PCF8574, symbol Interface_Expansion:PCF8574
- removed U7: DS18B20, Package_TO_SOT_THT:TO-92_Inline, symbol Sensor_Temperature:DS18B20
- added C2: 68nF, symbol Device:C
- added D1, D2, D3, D4: D, symbol Device:D
- added R13, R14, R15: 68R, symbol Device:R
- added U1: ESP32-DevKit-USB-C, ESP32:ESP32-DevKit-USB-C, symbol ESP32:ESP32-DevKit-USB-C
- added U7: AHT1x, Sensor:SHT1x, symbol Sensor:SHT1x
- R1, R2: value 4.7k -> 10k
- U8: value LM2596T-ADJ -> LM2596T-MODULE
- renumbered R8 to R3, R9 to R4, R10 to R5, R11 to R6, U11 to U9
Connections:
- net +5V is gone; now on net +3V3: U8.4 (FB)
- net +3V3: now also R7.2, C2.2, U1.16 (3V3), U7.4 (VDD); no longer R7.1
- net GND: now also U9.11, U9.13, U9.15, U9.9, C2.1, U1.14 (GND), U1.17 (GND), U7.1 (GND)
- net at R6.2, U9.7: now also D4.1 (K)
- net at U2.2 (DQ), U3.2 (DQ), U4.2 (DQ)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: now also R7.1, U1.13 (MTCK/GPIO13/ADC2_CH4); no longer R7.2, U6.2 (DQ)
- net at L3.1: now also C1.1, L1.1, L2.1, R1.2, R2.1, R13.1, R14.1, R15.1
- net at R3.2, U9.1: now also D1.1 (K)
- net at U9.2: now also D1.2 (A)
- net at L2.2: now also R14.2
- net at R5.2, U9.5: now also D3.1 (K)
- net at U9.6: now also D3.2 (A)
- net at L3.2: now also R15.2
- net at L1.2: now also R13.2
- net at R4.2, U9.3: now also D2.1 (K)
- net at U9.4: now also D2.2 (A)
- net at U9.8: now also D4.2 (A)
- new net: U1.29 (GPIO22), U7.2 (DATA)
- new net: U1.26 (GPIO21), U7.3 (SCK)
- now unconnected: U9.10, U9.12, U9.14, U9.16
Other:
- note added: "Burden resistors included in SCT sensors"
- moved on the sheet: C1, L1, L2, L3, R1, R2, R3, R4, R5, R6, R7, U2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
